File: stm32g474RET6 plytka/stm32g474RET6 plytka.kicad_sch (KiCad schematic)
At the start: 57 parts, among them IC1 STM32G484RET6, IC2 SN65HVD230DR, IC3 SN65HVD230DR, IC4 TPSM63603V3RDHR, IC5 ESP32-S3-WROOM-1-N8, J1 5055670431, J2 5055670631, J3 5055670631, J4 5055670631, SW1 SW_Push, SW2 SW_Push, SW3 SW_Push

Commit message: added test points
Parts:
- removed C11, C21: 1u, Capacitor_SMD:C_0603_1608Metric_Pad1.08x0.95mm_HandSolder, symbol Device:C
- removed C12, C15, C16, C19: 100n, Capacitor_SMD:C_0603_1608Metric_Pad1.08x0.95mm_HandSolder, symbol Device:C
- removed C18: 10u, Capacitor_SMD:C_0603_1608Metric_Pad1.08x0.95mm_HandSolder, symbol Device:C
- removed IC4: TPSM63603V3RDHR, Telemetry:TPSM63603EXTRDHR, symbol Telemetry:TPSM63603V3RDHR
- removed J1: 5055670431, Telemetry:CONN_505567_04_MOL, symbol Telemetry:5055670431
- removed J2, J3, J4: 5055670631, Telemetry:CONN_505567_06_MOL, symbol Telemetry:5055670631
- removed PS1: RPM5.0-3.0-CT, Telemetry:RPM5030CT, symbol Telemetry:RPM5.0-3.0-CT
- removed R1: 10R, Resistor_SMD:R_0603_1608Metric_Pad0.98x0.95mm_HandSolder, symbol Device:R
- removed R10, R8: 100k, Resistor_SMD:R_0603_1608Metric_Pad0.98x0.95mm_HandSolder, symbol Device:R
- removed R9: 20k, Resistor_SMD:R_0603_1608Metric_Pad0.98x0.95mm_HandSolder, symbol Device:R
- added C10, C14, C3, C8: 100n, Capacitor_SMD:C_0603_1608Metric_Pad1.08x0.95mm_HandSolder, symbol Device:C
- added C9: 1u, Capacitor_SMD:C_0603_1608Metric_Pad1.08x0.95mm_HandSolder, symbol Device:C
- added CAN1H1, CAN1L1, CAN2H1, CAN2L1, RX1, TX1: TestPoint, TestPoint:TestPoint_THTPad_1.5x1.5mm_Drill0.7mm, symbol Connector:TestPoint
- added J1, J2, J3, J4: MicroFit+ 6pin, Telemetry:CONN_2125280000_06_MOL, symbol Telemetry:MicroFit+ 6pin
- added R12, R7: 100R, Resistor_SMD:R_0603_1608Metric_Pad0.98x0.95mm_HandSolder, symbol Device:R
- C13: value 22u -> 100n
- IC4: renamed from IC1; footprint QFP50P1200X1200X160-64N -> Telemetry:QFP50P1200X1200X160-64N
- S1, S2: footprint CHS01TB -> Telemetry:CHS01TB
- renumbered C7 to C1, C2 to C11, C1 to C12, C4 to C15, C6 to C16, C8 to C2, C5 to C4, C3 to C5, C10 to C6, C17 to C7, D3 to D1, D1 to D3, IC5 to IC1, R13 to R1, R17 to R10, R16 to R11, R18 to R13, R19 to R14, R4 to R15, R6 to R16, R7 to R17, R3 to R2, R2 to R3, R14 to R4, R11 to R5, R15 to R6, R5 to R8, R12 to R9, SW2 to SW1, SW1 to SW2
Connections:
- net +3.3V: now also C11.1, C12.1, C13.1, IC4.29 (VDDA), C10.1, C14.1, C3.1, C8.1, C9.1, J2.2, J2.6, J4.6, R12.1, R7.1; no longer IC2.4 (R), IC3.4 (R), R11.1, R9.1
- net +5V: now also J3.6; no longer C13.1
- net GND: now also C10.2, C14.2, C3.2, C8.2, C9.2, J1.1, J2.1, J3.1, J4.1
- net SWCLK: now also J4.3
- net SWDIO: now also J4.2
- net CAN_1_Term: now reaches R3.1, S1.1 (COM)
- net CAN_1_N: now reaches IC2.6 (CANL), S1.2 (NO)
- net CAN_1_N: now also J1.5
- net NRST: now reaches C7.1, IC4.7 (PG10-NRST), R15.1, SW2.2
- net NRST: now also J4.4
- net at IC4.35 (PB13), R10.2: now also CAN2L1.1
- net CAN_2_Term: now reaches R2.1, S2.1 (COM)
- net CAN_2_P: now reaches IC3.7 (CANH), R2.2
- net CAN_2_P: now also J1.2
- net at D2.2 (A): now also J1.6
- net at IC1.27 (IO0), R4.1, SW1.1: now also J2.5
- net at R13.1: now also J3.2
- net at JP1.2 (B), R6.1: now also R12.2
- net at IC1.37 (TXD0), R6.2: now also J2.4, TX1.1
- net CAN_1_P: now reaches IC2.7 (CANH), R3.2
- net CAN_1_P: now also J1.4
- net at IC4.46 (PA12), R8.2: now also CAN1L1.1
- net at IC4.34 (PB12), R11.2: now also CAN2H1.1
- net CAN_2_N: now reaches IC3.6 (CANL), S2.2 (NO)
- net CAN_2_N: now also J1.3
- net at IC4.12 (PA0): now also J3.5
- net at IC4.13 (PA1): now also J3.4
- net at IC4.14 (PA2): now also J3.3
- net at IC4.45 (PA11), R9.2: now also CAN1H1.1
- net at JP2.2 (B), R5.1: now also R7.2
- net at IC1.36 (RXD0), R5.2: now also J2.3, RX1.1
- new net: IC3.4 (R), R11.1
- new net: IC2.4 (R), R9.1
- no-connect marks 79 -> 72
Other:
- added sheet Power Distribution (untitled.kicad_sch)
- moved on the sheet: C1, C11, C12, C15, C16, C2, C4, C5, C6, C7, D1, D2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
